File: regulator.kicad_sch (KiCad schematic)
At the start: 23 parts, among them U4 TPS63020DSJR, U5 MD53R33

Commit message: Added Graph & cleaned up title and layout
Other:
- company: FETfox -> github.com/FETfox/Li-Ion_Power_Module
- title: Li Lion Power Module -> Li Lion Power Module w/ Optional Fuel Gauge &CAN Bus
- moved on the sheet: C10, C11, C12, C25, C7, C8, C9, L1, LED3, R20, R21, R22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
