File: power_module.kicad_sch (KiCad schematic)
At the start: 0 parts

Commit message: Added labels and schematic PDF among other progress
Other:
- note added: "3v3"
- note added: "5V"

Commit message: Configured Varients
Other:
- note added: "5W/7W peak 2700 mAh Power Supply with USB Charging 3v3 or 5v w/ Optional Fuel Gauge & CAN Bus"
- note removed: "5W 2700 mAh Power Supply with USB Charging w/ Optional Fuel Gauge & CAN Bus"
Changed lines of the file:
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@@
 		)
 	)
-	(text "5W 2700 mAh Power Supply with USB Charging\nw/ Optional Fuel Gauge & CAN Bus"
+	(text "5W/7W peak 2700 mAh Power Supply with USB Charging\n3v3 or 5v w/ Optional Fuel Gauge & CAN Bus"
 		(exclude_from_sim no)
-		(at 13.208 13.716 0)
+		(at 85.09 19.812 0)
 		(effects
 			(font
@@
 				(bold yes)
 			)
-			(justify left top)
 		)
 	)

Commit message: Started work on PCB layout
Other:
- sheet Connectors renamed External Connectors
- sheet Power Regulator renamed Power Regulators
Changed lines of the file:
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@@
 			(color 0 0 0 0)
 		)
-		(property "Sheetname" "Power Regulator"
+		(property "Sheetname" "Power Regulators"
 			(at 104.14 108.5084 0)
 			(show_name no)
@@
 			(color 0 0 0 0)
 		)
-		(property "Sheetname" "Connectors"
+		(property "Sheetname" "External Connectors"
 			(at 104.14 128.8284 0)
 			(show_name no)
