File: power_module.kicad_pcb (KiCad board)
At the start: 2 copper layers, 124 parts, among them J1 UDPI, J2 OUT, J3 USB_C, J4 CELL, Q1 DMN2014LHAB-7, Q2 DMP3056L, U1 BQ24074RGT, U2 BQ29728, U3 BQ27427, U4 TPS63020DSJR, U5 MD53R33, U6 ATtiny3217, U7 MCP2515-xST, U8 SN65HVD230, Y1 16MHz

Commit message: Started work on PCB layout
Parts:
- removed the TP22 at (325.8, 278.1)
- added C25: 4.7nF, Capacitor_SMD:C_0603_1608Metric, F.Cu at (280.4, 489.1)
- added R26: 100k, Resistor_SMD:R_0603_1608Metric, F.Cu at (599.4, 492.9)
- added R51: 5.1k, Resistor_SMD:R_0603_1608Metric, F.Cu at (769.6, 293.9)
- added TP27: LDO_VIN, TestPoint:TestPoint_Pad_D1.0mm, F.Cu at (729.6, 36.8)
- added TP28: +3v3, TestPoint:TestPoint_Pad_D1.0mm, F.Cu at (577.6, 466.7)
- added TP30: LDO_VOUT, TestPoint:TestPoint_Pad_D1.0mm, F.Cu at (737.2, 36.8)
- added TP31: NTC, TestPoint:TestPoint_Pad_D1.0mm, F.Cu at (403.4, 392.4)
- added TP32: MCU_VCC, TestPoint:TestPoint_Pad_D1.0mm, F.Cu at (397.0, 391.9)
- added TP33: SPI_MOSI, TestPoint:TestPoint_Pad_D1.0mm, F.Cu at (106.3, 437.8)
- added TP34: SPI_MISO, TestPoint:TestPoint_Pad_D1.0mm, F.Cu at (106.3, 440.8)
- added TP35: CAN_CS, TestPoint:TestPoint_Pad_D1.0mm, F.Cu at (106.3, 443.9)
- added TP36: SPI_SCK, TestPoint:TestPoint_Pad_D1.0mm, F.Cu at (106.3, 446.9)
- added TP37: CAN_RESET, TestPoint:TestPoint_Pad_D1.0mm, F.Cu at (109.4, 437.8)
- added TP38: CAN_INT, TestPoint:TestPoint_Pad_D1.0mm, F.Cu at (109.4, 440.8)
- added TP39: TXCAN, TestPoint:TestPoint_Pad_D1.0mm, F.Cu at (273.9, 495.4)
- added TP40: RXCAN, TestPoint:TestPoint_Pad_D1.0mm, F.Cu at (273.9, 498.5)
- added TP41: VREF, TestPoint:TestPoint_Pad_D1.0mm, F.Cu at (276.9, 489.4)
- added TP42: CANH, TestPoint:TestPoint_Pad_D1.0mm, F.Cu at (276.9, 492.4)
- added TP43: CANL, TestPoint:TestPoint_Pad_D1.0mm, F.Cu at (276.9, 495.4)
- added TP44: ADC_CC2, TestPoint:TestPoint_Pad_D1.0mm, F.Cu at (766.4, 291.5)
- added TP45: ADC_CC1, TestPoint:TestPoint_Pad_D1.0mm, F.Cu at (766.4, 294.0)
- BT1: footprint BatterySleds:BatteryHolder_HAN_BH-18650-1 -> footprints:BatteryHolder_HAN_BH-18650-1
- C11: value 10uF -> 22uF; footprint Capacitor_SMD:C_0603_1608Metric -> Capacitor_SMD:C_0805_2012Metric
- C13: value 22uF -> 10uF; footprint Capacitor_SMD:C_0805_2012Metric -> Capacitor_SMD:C_0603_1608Metric
- C14: value 100nF -> 22uF; footprint Capacitor_SMD:C_0603_1608Metric -> Capacitor_SMD:C_0805_2012Metric
- C16: value 10nF -> 100nF
- C17: value 10pF -> 10nF
- C19: value 4.7uF -> 10pF; footprint Capacitor_SMD:C_0805_2012Metric -> Capacitor_SMD:C_0603_1608Metric
- C20: value 100nF -> 4.7uF; footprint Capacitor_SMD:C_0603_1608Metric -> Capacitor_SMD:C_0805_2012Metric
- C22: value 100pF -> 100nF
- C24: value 4.7nF -> 100pF
- J3: renamed from J1; value UDPI -> Conn_02x03_Pogo
- J4: value CELL -> JST PH B4B
- Q1: footprint DFN:U-DFN2030-6 -> footprints:U-DFN2030-6
- R10: renamed from R6; value 0R -> 1.1k; footprint Resistor_SMD:R_0805_2012Metric -> Resistor_SMD:R_0603_1608Metric
- R18: renamed from R8; value 1.1k -> 0R; footprint Resistor_SMD:R_0603_1608Metric -> Resistor_SMD:R_0805_2012Metric
- R19: value 0R -> 10k; footprint Resistor_SMD:R_1206_3216Metric -> Resistor_SMD:R_0603_1608Metric
- R20: value 100R -> 0R; footprint Resistor_SMD:R_0603_1608Metric -> Resistor_SMD:R_1206_3216Metric
- R21: renamed from R23; value 100k -> 0R; footprint Resistor_SMD:R_0603_1608Metric -> Resistor_SMD:R_1206_3216Metric
- R22: renamed from R25; value 137k -> 1.2M
- R23: renamed from R26; value 0R -> 137k; footprint Resistor_SMD:R_1206_3216Metric -> Resistor_SMD:R_0603_1608Metric
- R24: renamed from R27; footprint Resistor_SMD:R_0805_2012Metric -> Resistor_SMD:R_1206_3216Metric
- R27: renamed from R24; value 1.2M -> 100k
- R28: renamed from R21; value 10k -> 100R
- R29: renamed from R22; value 0R -> 10k; footprint Resistor_SMD:R_1206_3216Metric -> Resistor_SMD:R_0603_1608Metric
- R30: renamed from R29; value 1R -> 0R; footprint Resistor_SMD:R_0603_1608Metric -> Resistor_SMD:R_0805_2012Metric
- R31: renamed from R30; value 5.1k -> 1R
- R33: renamed from R31; value 5.1k -> 0R; footprint Resistor_SMD:R_0603_1608Metric -> Resistor_SMD:R_0805_2012Metric
- R34: renamed from R32; value 5.1k -> 100R
- R35: renamed from R34; value 10k -> 5.1k
- R36: renamed from R35; value 10k -> 5.1k
- R37: renamed from R36; value 0R -> 5.1k; footprint Resistor_SMD:R_0805_2012Metric -> Resistor_SMD:R_0603_1608Metric
- R39: renamed from R38; value 100R -> 10k
- R40: renamed from R39; value 0R -> 10k; footprint Resistor_SMD:R_0805_2012Metric -> Resistor_SMD:R_0603_1608Metric
- R43: renamed from R42; value 100R -> 0R; footprint Resistor_SMD:R_0603_1608Metric -> Resistor_SMD:R_0805_2012Metric
- R45: renamed from R44; value 10k -> 100R
- R46: renamed from R45; value 0R -> 10k; footprint Resistor_SMD:R_0805_2012Metric -> Resistor_SMD:R_0603_1608Metric
- R47: renamed from R46; value 60.4R -> 0R; footprint Resistor_SMD:R_0603_1608Metric -> Resistor_SMD:R_0805_2012Metric
- R49: renamed from R48; value 5.1k -> 60.4R
- R5: renamed from R17; value 100k -> 0R; footprint Resistor_SMD:R_0603_1608Metric -> Resistor_SMD:R_1206_3216Metric
- R6: renamed from R18; value 10k -> 100k
- TP1: renamed from TP10; value SRX -> BAT
- TP10: renamed from TP13; value I2C_SCL -> TS
- TP11: renamed from TP4; value EN1 -> TMR
- TP12: renamed from TP24; value TXCAN -> +Pack
- TP13: renamed from TP14; value I2C_SDA -> CHG_OUT
- TP14: renamed from TP15; value FG_BATT -> SRX
- TP15: renamed from TP5; value 5V -> ILIM
- TP16: value +Pack -> BIN
- TP17: renamed from TP7; value CHG_PGOOD -> ITERM
- TP18: renamed from TP19; value NTC -> FG_GPOUT
- TP19: renamed from TP20; value SPI_MOSI -> I2C_SCL
- TP2: renamed from TP17; value REG_OUT -> +Cell
- TP20: renamed from TP21; value SPI_MISO -> I2C_SDA
- TP21: renamed from TP3; value CE -> EN2
- TP22: renamed from TP23; value SPI_SCK -> FG_VDD
- TP23: renamed from TP6; value GND -> EN1
- TP24: renamed from TP26; value VREF -> REG_Vina
- TP25: renamed from TP27; value CANH -> REG_VIN
- TP26: renamed from TP28; value CANL -> REG_OUT
- TP29: renamed from TP25; value RXCAN -> REG_PGOOD
- TP3: renamed from TP18; value +3v3 -> -Cell
- TP4: renamed from TP1; value EN2 -> CE
- TP5: renamed from TP8; value CHG -> 5V
- TP6: renamed from TP9; value CHG_OUT -> GND
- TP8: renamed from TP11; value +Cell -> CHG_PGOOD
- TP9: renamed from TP12; value -Cell -> CHG
- U1: renamed from U2; footprint Package_SON:WSON-6_1.5x1.5mm_P0.5mm -> footprints:WSON-6_1.5x1.5mm_P0.5mm
- U2: renamed from U1; footprint Package_DFN_QFN:VQFN-16-1EP_3x3mm_P0.5mm_EP1.6x1.6mm -> footprints:VQFN-16-1EP_3x3mm_P0.5mm_EP1.6x1.6mm_ThermalVias
- U3: footprint BGA:IC_BQ27427YZFR -> footprints:BQ27427
- U4: footprint vson:IC_TPS63020DSJR -> footprints:IC_TPS63020DSJR
- moved J2 535.5 mm to (874.7, 231.2)
- moved J4 535.5 mm to (874.7, 237.7)
- moved R31 442.0 mm to (738.1, 41.9), turned to 180 degrees
- moved R30 441.7 mm to (734.7, 35.8), turned to 90 degrees
- moved C13 441.5 mm to (738.0, 40.0)
- moved U5 427.3 mm to (733.6, 41.0)
- moved R25 427.2 mm to (732.2, 35.8), turned to 90 degrees
- moved J1 427.2 mm to (770.8, 300.1)
- moved D1 426.1 mm to (759.0, 153.2)
- moved C12 426.0 mm to (728.8, 40.0), turned to 180 degrees
- moved TVS2 424.4 mm to (778.3, 292.7), turned to 180 degrees
- moved J3 421.9 mm to (760.6, 157.8)
- moved R50 420.5 mm to (772.2, 293.9), turned to -90 degrees
- moved R28 322.7 mm to (608.5, 504.2)
- moved TP29 320.6 mm to (575.4, 483.0)
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- renumbered C3 to C1, C1 to C2, C2 to C3, J3 to J1, R10 to R1, R14 to R11, R9 to R12, R2 to R13, R3 to R14, R7 to R17, R13 to R2, R28 to R25, R1 to R3, R33 to R32, R37 to R38, R40 to R41, R41 to R42, R43 to R44, R47 to R48, R49 to R50, R11 to R7, R5 to R8, R12 to R9, TP2 to TP7
Connections:
- net /Connectors/UART_RX renamed /External Connectors/UART_RX
- net /Connectors/UART_TX renamed /External Connectors/UART_TX
- net /Power Regulator/SW1 renamed /Power Regulators/SW1
- net /Power Regulator/SW2 renamed /Power Regulators/SW2
- net Net-(D1-A) renamed /External Connectors/UPDI_VCC
- net Net-(LED1-A) renamed /Battery Management/LED1_R
- net Net-(LED2-A) renamed /Battery Management/LED2_R
- C11 pad 1: /Power Regulator/LDO_VIN -> REG_VOUT
- C12 pad 1: /Power Regulator/LDO_VOUT -> /Power Regulators/LDO_VIN
- C12 pad 2: Net-(C12-Pad2) -> GND
- C13 pad 1: GND -> /Power Regulators/LDO_VOUT
- C13 pad 2: /MCU/MCU_VCC -> /Power Regulators/LDO_SNUB
- C15 pad 2: +3V3 -> /MCU/MCU_VCC
- C17 pad 2: /CAN Bus/OSC1 -> +3V3
- C18 pad 2: Net-(C18-Pad2) -> /CAN Bus/OSC1
- C19 pad 2: +3V3 -> /CAN Bus/OSC_TUNE
- C21 pad 1: Net-(U8-D) -> /CAN Bus/CANTRANS_D
- C22 pad 1: /CAN Bus/CANH -> GND
- C22 pad 2: GND -> +3V3
- C23 pad 1: /CAN Bus/CANL -> GND
- C23 pad 2: GND -> /CAN Bus/CANH
- C24 pad 1: /CAN Bus/Vref -> /CAN Bus/CANL
- C7 pad 1: /Power Regulator/Vina -> /Power Regulators/Vina
- C8 pad 1: /Power Regulator/REG_VIN -> /Power Regulators/REG_VIN
- C9 pad 1: REG_VOUT -> /Power Regulators/REG_VIN
- J1 pad A5: /Connectors/ADC_CC1 -> /External Connectors/ADC_CC1
- J1 pad B5: /Connectors/ADC_CC2 -> /External Connectors/ADC_CC2
- J3 pad 6: /Connectors/UDPI -> /External Connectors/UPDI
- LED3 pad 1: /Power Regulator/REG_PGOOD -> /Power Regulators/REG_PGOOD
- LED3 pad 2: Net-(LED3-A) -> /Power Regulators/LED3_R
- Q2 pad 1: Net-(Q2-G) -> /Battery Management/POL_GATE
- R10 pad 1: /Battery Management/CHG_EN1 -> /Battery Management/ILIM
- R10 pad 2: +5V -> GND
- R17 pad 1: GND -> /Battery Management/CHG_EN1
- R17 pad 2: /Battery Management/CHG_EN1 -> +5V
- R18 pad 1: /Battery Management/ILIM -> GND
- R18 pad 2: GND -> /Battery Management/CHG_EN1
- R19 pad 1: SRX -> /Battery Management/CHG_PGOOD
- R19 pad 2: +PACK -> VDC
- R20 pad 1: Net-(LED3-A) -> SRX
- R20 pad 2: +3V3 -> +PACK
- R21 pad 1: /MCU/PS -> VDC
- R21 pad 2: GND -> /Power Regulators/REG_VIN
- R22 pad 1: /Power Regulator/FB -> REG_VOUT
- R22 pad 2: GND -> /Power Regulators/FB
- R23 pad 1: REG_VOUT -> /Power Regulators/FB
- R23 pad 2: +3V3 -> GND
- R24 pad 1: /Power Regulator/LDO_VIN -> REG_VOUT
- R24 pad 2: REG_VOUT -> +3V3
- R25 pad 1: /Power Regulator/LDO_VOUT -> /Power Regulators/LDO_VIN
- R25 pad 2: +3V3 -> REG_VOUT
- R27 pad 1: REG_VOUT -> /MCU/PS
- R27 pad 2: /Power Regulator/FB -> GND
- R28 pad 1: /Power Regulator/REG_PGOOD -> /Power Regulators/LED3_R
- R29 pad 1: VDC -> /Power Regulators/REG_PGOOD
- R29 pad 2: /Power Regulator/REG_VIN -> +3V3
- R30 pad 1: Net-(C12-Pad2) -> /Power Regulators/LDO_VOUT
- R30 pad 2: GND -> +3V3
- R31 pad 1: /Battery Management/FG_GPOUT -> /Power Regulators/LDO_SNUB
- R31 pad 2: /MCU/MCU_VCC -> GND
- R32 pad 1: /MCU/MCU_VCC -> /MCU/NTC_MCU
- R32 pad 2: /CAN Bus/CAN_CS -> /MCU/MCU_VCC
- R33 pad 1: /Battery Management/I2C_SDA -> +3V3
- R34 pad 1: /MCU/MCU_VCC -> /MCU/UPDI_MCU
- R34 pad 2: /Battery Management/I2C_SCL -> /MCU/UPDI
- R35 pad 1: /MCU/MCU_VCC -> /Battery Management/FG_GPOUT
- R35 pad 2: /CAN Bus/CAN_RESET -> /MCU/MCU_VCC
- R36 pad 1: /CAN Bus/CAN_INT -> /Battery Management/I2C_SDA
- R37 pad 1: +3V3 -> /MCU/MCU_VCC
- R37 pad 2: /MCU/MCU_VCC -> /Battery Management/I2C_SCL
- R38 pad 1: /MCU/NTC_MCU -> /MCU/MCU_VCC
- R38 pad 2: /MCU/MCU_VCC -> /CAN Bus/CAN_CS
- R39 pad 1: /MCU/UPDI_MCU -> /MCU/MCU_VCC
- R39 pad 2: /Connectors/UDPI -> /CAN Bus/CAN_RESET
- R40 pad 1: +3V3 -> /CAN Bus/CAN_INT
- R40 pad 2: Net-(U7-VDD) -> /MCU/MCU_VCC
- R41 pad 1: Net-(C18-Pad2) -> +3V3
- R41 pad 2: /CAN Bus/OSC2 -> /CAN Bus/CAN_CTRL_VDD
- R42 pad 1: /CAN Bus/OSC1 -> /CAN Bus/OSC_TUNE
- R43 pad 1: /CAN Bus/TXCAN -> /CAN Bus/OSC1
- R43 pad 2: Net-(U8-D) -> /CAN Bus/OSC2
- R44 pad 1: Net-(U8-R) -> /CAN Bus/TXCAN
- R44 pad 2: /CAN Bus/RXCAN -> /CAN Bus/CANTRANS_D
- R45 pad 1: GND -> /CAN Bus/CANTRANS_R
- R45 pad 2: /CAN Bus/Rs -> /CAN Bus/RXCAN
- R46 pad 1: +3V3 -> GND
- R46 pad 2: Net-(U8-VCC) -> /CAN Bus/Rs
- R47 pad 1: /CAN Bus/Vref -> +3V3
- R47 pad 2: /CAN Bus/CANH -> /CAN Bus/CAN_TRANS_VCC
- R48 pad 1: /CAN Bus/CANL -> /CAN Bus/Vref
- R48 pad 2: /CAN Bus/Vref -> /CAN Bus/CANH
- R49 pad 1: GND -> /CAN Bus/CANL
- R49 pad 2: /Connectors/ADC_CC2 -> /CAN Bus/Vref
- R5 pad 1: -CELL -> +CELL
- R5 pad 2: Net-(Q2-G) -> +PACK
- R50 pad 2: /Connectors/ADC_CC1 -> /External Connectors/ADC_CC2
- R6 pad 1: /Battery Management/CHG_PGOOD -> -CELL
- R6 pad 2: VDC -> /Battery Management/POL_GATE
- TP1 pad 1: SRX -> /Battery Management/BAT
- TP10 pad 1: /Battery Management/I2C_SCL -> /Battery Management/TS
- TP11 pad 1: /Battery Management/CHG_EN1 -> /Battery Management/TMR
- TP12 pad 1: /CAN Bus/TXCAN -> +PACK
- TP13 pad 1: /Battery Management/I2C_SDA -> VDC
- TP14 pad 1: +PACK -> SRX
- TP15 pad 1: +5V -> /Battery Management/ILIM
- TP16 pad 1: +PACK -> /Battery Management/BIN
- TP17 pad 1: /Battery Management/CHG_PGOOD -> /Battery Management/ITERM
- TP18 pad 1: /MCU/NTC_MCU -> /Battery Management/FG_GPOUT
- TP19 pad 1: /CAN Bus/SPI_MOSI -> /Battery Management/I2C_SCL
- TP2 pad 1: REG_VOUT -> +CELL
- TP20 pad 1: /CAN Bus/SPI_MISO -> /Battery Management/I2C_SDA
- TP21 pad 1: /Battery Management/CE -> /Battery Management/CHG_EN2
- TP22 pad 1: /CAN Bus/SPI_SCK -> /Battery Management/FG_VDD
- TP23 pad 1: GND -> /Battery Management/CHG_EN1
- TP24 pad 1: /CAN Bus/Vref -> /Power Regulators/Vina
- TP25 pad 1: /CAN Bus/CANH -> /Power Regulators/REG_VIN
- TP26 pad 1: /CAN Bus/CANL -> REG_VOUT
- TP29 pad 1: /CAN Bus/RXCAN -> /Power Regulators/REG_PGOOD
- TP3 pad 1: +3V3 -> -CELL
- TP4 pad 1: /Battery Management/CHG_EN2 -> /Battery Management/CE
- TP5 pad 1: /Battery Management/CHG -> +5V
- TP6 pad 1: VDC -> GND
- TP8 pad 1: +CELL -> /Battery Management/CHG_PGOOD
- TP9 pad 1: -CELL -> /Battery Management/CHG
- U2 pad 3: /Battery Management/CHG -> SRX
- U4 pad 1: /Power Regulator/Vina -> /Power Regulators/Vina
- U4 pad 10: /Power Regulator/REG_VIN -> /Power Regulators/REG_VIN
- U4 pad 11: /Power Regulator/REG_VIN -> /Power Regulators/REG_VIN
- U4 pad 12: /Power Regulator/Vina -> /Power Regulators/Vina
- U4 pad 14: /Power Regulator/REG_PGOOD -> /Power Regulators/REG_PGOOD
- U4 pad 3: /Power Regulator/FB -> /Power Regulators/FB
- U5 pad 1: /Power Regulator/LDO_VIN -> /Power Regulators/LDO_VIN
- U5 pad 3: /Power Regulator/LDO_VIN -> /Power Regulators/LDO_VIN
- U5 pad 5: /Power Regulator/LDO_VOUT -> /Power Regulators/LDO_VOUT
- U6 pad 2: /Power Regulator/REG_PGOOD -> /Power Regulators/REG_PGOOD
- U6 pad 21: /Connectors/ADC_CC1 -> /External Connectors/ADC_CC1
- U6 pad 22: /Connectors/ADC_CC2 -> /External Connectors/ADC_CC2
- U7 pad 20: Net-(U7-VDD) -> /CAN Bus/CAN_CTRL_VDD
- U8 pad 1: Net-(U8-D) -> /CAN Bus/CANTRANS_D
- U8 pad 3: Net-(U8-VCC) -> /CAN Bus/CAN_TRANS_VCC
- U8 pad 4: Net-(U8-R) -> /CAN Bus/CANTRANS_R
- Y1 pad 3: Net-(C18-Pad2) -> /CAN Bus/OSC_TUNE
Routing:
- net GND: track 0.00 -> 49.1 mm, vias 0 -> 40
- net +5V: track 0.00 -> 32.3 mm
- net /MCU/MCU_VCC: track 0.00 -> 29.9 mm, vias 0 -> 4
- net VDC: track 0.00 -> 29.9 mm
- net /Battery Management/ADC_ISET: track 0.00 -> 23.6 mm
- net /Battery Management/CHG_PGOOD: track 0.00 -> 20.5 mm
- net /Battery Management/TS: track 0.00 -> 19.0 mm
- net +PACK: track 0.00 -> 16.8 mm
- net SRX: track 0.00 -> 16.3 mm
- net /External Connectors/ADC_CC2: track 0.00 -> 15.9 mm
- net /Power Regulators/LDO_VIN: track 0.00 -> 15.1 mm
- net /Battery Management/CE: track 0.00 -> 15.0 mm
- net /Battery Management/ITERM: track 0.00 -> 14.7 mm
- net /External Connectors/ADC_CC1: track 0.00 -> 14.0 mm
- net /Power Regulators/REG_PGOOD: track 0.00 -> 13.2 mm, vias 0 -> 1
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- added copper zone on F.Cu, net /Power Regulators/REG_VIN
- added copper zone on F.Cu, net GND
- added copper zone on F.Cu, net REG_VOUT
Other:
- copper layers 2 -> 4

Commit message: Initial commit
Parts:
- removed TP29: REG_PGOOD, TestPoint:TestPoint_Pad_D1.0mm
- added NT1: NetTie_2, NetTie:NetTie-2_SMD_Pad2.0mm, F.Cu at (230.8, 330.1)
- J2: value OUT -> JST_PH
- J4: value JST PH B4B -> JST_PH
- Q2: value DMP3056L -> DMP2008UFG-7; footprint Package_TO_SOT_SMD:SOT-23 -> Package_SON:Diodes_PowerDI3333-8
- moved J1 598.6 mm to (172.7, 277.5)
- moved R51 598.6 mm to (171.5, 271.4)
- moved TP44 598.6 mm to (168.3, 268.9)
- moved TP45 598.6 mm to (168.3, 271.4)
- moved TVS2 598.6 mm to (180.1, 270.2)
- moved R50 598.6 mm to (174.0, 271.4)
- moved C13 541.1 mm to (258.1, 290.1)
- moved R30 541.1 mm to (254.8, 285.9)
- moved TP27 541.1 mm to (249.7, 286.9)
- moved TP30 541.1 mm to (257.4, 286.9)
- moved U5 541.1 mm to (253.7, 291.1)
- moved R25 541.1 mm to (252.3, 285.9)
- moved R31 541.1 mm to (258.2, 292.0)
- moved C12 540.8 mm to (249.3, 290.1)
- moved J3 513.5 mm to (278.8, 335.4), turned to -90 degrees
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Connections:
- C16 pad 2: +3V3 -> /CAN Bus/CAN_CTRL_VDD
- C17 pad 2: +3V3 -> /CAN Bus/CAN_CTRL_VDD
- C20 pad 2: +3V3 -> /CAN Bus/CAN_TRANS_VCC
- C22 pad 2: +3V3 -> /CAN Bus/CAN_TRANS_VCC
- Q2 pad 1: /Battery Management/POL_GATE -> +PACK
- Q2 pad 3: +CELL -> +PACK
- U4 pad 1: /Power Regulators/Vina -> unconnected-(U4-VINA-Pad1)
- U4 pad 12: /Power Regulators/Vina -> /Power Regulators/REG_EN
Routing:
- net GND: track 49.1 -> 106.3 mm, vias 40 -> 47
- net /Power Regulators/Vina: track 7.41 -> 29.8 mm
- net +3V3: track 0.00 -> 20.4 mm
- net /CAN Bus/CAN_CTRL_VDD: track 0.00 -> 19.3 mm
- net /CAN Bus/OSC1: track 0.00 -> 14.8 mm
- net /CAN Bus/CAN_INT: track 5.15 -> 19.7 mm
- net /CAN Bus/OSC_TUNE: track 0.00 -> 14.3 mm
- net /CAN Bus/SPI_SCK: track 6.08 -> 18.8 mm
- net /CAN Bus/CANH: track 0.00 -> 11.4 mm
- net /CAN Bus/SPI_MOSI: track 5.45 -> 16.7 mm
- net /CAN Bus/CANL: track 0.00 -> 11.0 mm
- net /CAN Bus/OSC2: track 0.00 -> 10.8 mm
- net /CAN Bus/CAN_TRANS_VCC: track 0.00 -> 9.53 mm
- net /CAN Bus/SPI_MISO: track 5.34 -> 14.8 mm
- net /CAN Bus/CAN_CS: track 5.79 -> 13.5 mm
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- added copper zone on F.Cu, net +CELL
- added copper zone on F.Cu, net +PACK
- added copper zone on F.Cu, net /Power Regulators/SW1
- added copper zone on F.Cu, net /Power Regulators/SW2
Other:
- board text added: "3v3 LDO"
- board text added: "5V DC IN"
- board text added: "CANBUS CONTROLLER"
- board text added: "CELL MANAGMENT"
- board text added: "MAIN REGULATOR"
- board text added: "MCU"
- board text added: "NOTE! CAN needs inducdance matching diff pair!"
- board text added: "UPDI Connector"
- board text added: "USB-C PORT"

Commit message: Arranging Passives more effeciently
Parts:
- moved TP22 361.0 mm to (152.9, 291.6), turned to 90 degrees
- moved TP19 358.6 mm to (152.9, 294.1), turned to 90 degrees
- moved C5 356.5 mm to (156.2, 292.6), turned to 90 degrees
- moved TP20 356.3 mm to (152.9, 296.6), turned to 90 degrees
- moved TP18 354.0 mm to (152.9, 299.2), turned to 90 degrees
- moved C6 353.3 mm to (158.7, 293.5), turned to 0 degrees
- moved TP16 351.7 mm to (152.9, 301.7), turned to 90 degrees
- moved U3 351.5 mm to (157.4, 296.6), turned to 90 degrees
- moved R20 347.4 mm to (161.3, 296.6), turned to 90 degrees
- moved R11 347.3 mm to (158.2, 299.2), turned to 0 degrees
- moved Q2 340.5 mm to (243.2, 307.2), turned to -90 degrees
- moved TP2 339.6 mm to (250.2, 308.8), turned to -90 degrees
- moved R5 337.5 mm to (246.3, 305.9), turned to 90 degrees
- moved TP12 336.3 mm to (250.2, 306.2), turned to -90 degrees
- moved R6 334.2 mm to (243.1, 303.5), turned to 180 degrees
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Routing:
- net /Battery Management/ADC_ISET: track 27.4 -> 19.1 mm
- net /Battery Management/I2C_SDA: track 12.5 -> 7.59 mm
- net /Battery Management/FG_GPOUT: track 12.9 -> 8.12 mm
- net /Battery Management/FG_VDD: track 11.9 -> 7.68 mm
- net /MCU/MCU_VCC: track 29.3 -> 25.4 mm, vias 4 -> 3
- net /CAN Bus/CAN_RESET: track 13.6 -> 9.89 mm
- net /Battery Management/I2C_SCL: track 11.0 -> 7.34 mm
- net +CELL: track 5.59 -> 2.23 mm
- net /Battery Management/BIN: track 11.0 -> 7.81 mm
- net /Battery Management/CHG_PGOOD: track 20.5 -> 23.3 mm
- net /Battery Management/POL_GATE: track 4.74 -> 2.21 mm
- net /CAN Bus/CAN_INT: track 19.7 -> 17.6 mm
- net /MCU/UPDI_MCU: track 3.66 -> 2.14 mm
- net /CAN Bus/CAN_CS: track 13.5 -> 12.0 mm
- net -CELL: track 16.9 -> 15.7 mm
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Other:
- board text added: "Fuel Guage"
- board text added: "Polarity Protection"
- board text removed: "5V DC IN"
